Commit message: Add files via upload

File: description/robot_core.xacro (robot description, xacro)
@@ -7,8 +7,8 @@
     <xacro:property name="wheel_mass" value="${track_mass/3}"/>
     <xacro:property name="min_depth" value="0.001"/>
-    <xacro:property name="mu1" value="1.5"/>
-    <!-- Было 1 -->
-    <xacro:property name="mu2" value="1.0"/>
+    <xacro:property name="mu1" value="0.7"/>
+    <xacro:property name="mu2" value="0.7"/>
     <xacro:property name="kp" value="1000000"/>
+    <!-- <xacro:property name="kd" value="100"/> -->
     <!-- <xacro:property name="kd" value="100"/> -->
 <!-- MATERIALS -->
@@ -49,5 +49,5 @@
             <origin xyz="0 0 0" rpy="0 0 ${pi}"/>
             <geometry>
-                <mesh filename="file://$(find my_bot)/meshes/2-Chassis.stl" />
+                <mesh filename="file://$(find test_bot)/meshes/2-Chassis.stl" />
             </geometry>
             <material name="white"/>
