Commit message: workable movement

File: description/robot.urdf.xacro (robot description, xacro)
@@ -8,3 +8,4 @@
     </xacro:if>
     <xacro:include filename="lidar.xacro" />
+    <xacro:include filename="depth_camera.xacro" />
 </robot>

File: description/ros2_control.xacro (robot description, xacro)
@@ -25,4 +25,14 @@
             <xacro:wheel_joint name="right_wheel2_joint"/>
             <xacro:wheel_joint name="right_wheel3_joint"/>
+            <joint name="forward_track_joint">
+                <command_interface name="position"/>
+                <state_interface name="position"/>
+                <state_interface name="velocity"/>
+            </joint>
+            <joint name="backward_track_joint">
+                <command_interface name="position"/>
+                <state_interface name="position"/>
+                <state_interface name="velocity"/>
+            </joint>
         </ros2_control>
     </xacro:if>
